File: ESP32-S3/ESP32-S3.kicad_pcb (KiCad board)
At the start: 2 copper layers, 4 parts, among them J1 Conn_01x08, J2 FlySky Receiver, J3 Conn_01x08, U1 ESP32-S3-DevKitC-1-N32R16V

Commit message: Add files via upload
Parts:
- added C3: 1uF, Capacitor_THT:CP_Radial_D5.0mm_P2.00mm, F.Cu at (137.2, 154.3)
- added C4: 1uF, Capacitor_THT:CP_Radial_D5.0mm_P2.00mm, F.Cu at (137.2, 160.8)
- added Q3: BC183, Package_TO_SOT_THT:TO-92_Inline, F.Cu at (136.8, 167.4)
- added Q4: BC183, Package_TO_SOT_THT:TO-92_Inline, F.Cu at (136.8, 173.1)
- added R10: 2.2k, Resistor_THT:R_Axial_DIN0207_L6.3mm_D2.5mm_P10.16mm_Horizontal, F.Cu at (123.1, 165.2)
- added R11: 680, Resistor_THT:R_Axial_DIN0207_L6.3mm_D2.5mm_P10.16mm_Horizontal, F.Cu at (123.1, 169.2)
- added R12: 1k, Resistor_THT:R_Axial_DIN0207_L6.3mm_D2.5mm_P10.16mm_Horizontal, F.Cu at (123.1, 173.3)
- added R7: 2.2k, Resistor_THT:R_Axial_DIN0207_L6.3mm_D2.5mm_P10.16mm_Horizontal, F.Cu at (123.1, 153.0)
- added R8: 680, Resistor_THT:R_Axial_DIN0207_L6.3mm_D2.5mm_P10.16mm_Horizontal, F.Cu at (123.1, 157.1)
- added R9: 1k, Resistor_THT:R_Axial_DIN0207_L6.3mm_D2.5mm_P10.16mm_Horizontal, F.Cu at (123.1, 161.1)
Connections:
- U1 pad J115: Net-(J3-Pin_2) -> Net-(U1-5)
- U1 pad J120: Net-(J3-Pin_7) -> Net-(U1-17)
